Commit message: test_env.py - basic open_manipulator loading

File: assets/open_manipulator/open_manipulator_robot.urdf (robot description, URDF)
Before this commit: robot open_manipulator, 9 links, 8 joints
Links:
- link gripper_link: geometry collision mesh filename=./meshes/chain_link_grip_l.obj scale=0.001 0.001 0.001; visual mesh filename=./meshes/chain_link_grip_l.obj scale=0.001 0.001 0.001
- link gripper_link_sub: geometry collision mesh filename=./meshes/chain_link_grip_r.obj scale=0.001 0.001 0.001; visual mesh filename=./meshes/chain_link_grip_r.obj scale=0.001 0.001 0.001
- link link1: geometry collision mesh filename=./meshes/chain_link1.obj scale=0.001 0.001 0.001; visual mesh filename=./meshes/chain_link1.obj scale=0.001 0.001 0.001
- link link2: geometry collision mesh filename=./meshes/chain_link2.obj scale=0.001 0.001 0.001; visual mesh filename=./meshes/chain_link2.obj scale=0.001 0.001 0.001
- link link3: geometry collision mesh filename=./meshes/chain_link3.obj scale=0.001 0.001 0.001; visual mesh filename=./meshes/chain_link3.obj scale=0.001 0.001 0.001
- link link4: geometry collision mesh filename=./meshes/chain_link4.obj scale=0.001 0.001 0.001; visual mesh filename=./meshes/chain_link4.obj scale=0.001 0.001 0.001
- link link5: geometry collision mesh filename=./meshes/chain_link5.obj scale=0.001 0.001 0.001; visual mesh filename=./meshes/chain_link5.obj scale=0.001 0.001 0.001

Commit message: basic static omx env setup with table and cube

File: assets/open_manipulator/open_manipulator_robot.urdf (robot description, URDF)
Before this commit: robot open_manipulator, 9 links, 8 joints
Links:
- removed link world
- link end_effector_link: mass 1.0e-03 -> 1.0e-06; geometry visual box size=0.005 0.005 0.005
Joints:
- removed joint world_fixed

Commit message: joint_position_control basic done

File: assets/open_manipulator/open_manipulator_robot.urdf (robot description, URDF)
Before this commit: robot open_manipulator, 8 links, 7 joints
Links:
- link end_effector_link: mass 1.0e-06 -> None
